File: KiCad/ArxRP2040Devboard/ArxRP2040Devboard.kicad_pcb (KiCad board)
At the start: 2 copper layers, 21 x 51 mm, 3 parts, among them U1 NCP1117-1.5_SOT223, U2 RP2040, U3 W25Q128JVS

Commit message: schematics
Parts:
- removed U3: W25Q128JVS, Package_SO:SOIC-8_5.3x5.3mm_P1.27mm
- added C1: 1uF, Capacitor_SMD:C_0402_1005Metric, F.Cu at (135.5, 108.3)
- added C10: 1uF, Capacitor_SMD:C_0402_1005Metric, F.Cu at (132.5, 117.8)
- added C11: 0.1uF, Capacitor_SMD:C_0402_1005Metric, F.Cu at (132.5, 104.0)
- added C12: 0.1uF, Capacitor_SMD:C_0402_1005Metric, F.Cu at (131.5, 104.2)
- added C13: 10uF, Capacitor_SMD:C_0603_1608Metric, F.Cu at (126.7, 88.7)
- added C14: 10uF, Capacitor_SMD:C_0603_1608Metric, F.Cu at (126.6, 94.3)
- added C15: 33pF, Capacitor_SMD:C_0402_1005Metric, F.Cu at (124.8, 120.5)
- added C16: 33pF, Capacitor_SMD:C_0402_1005Metric, F.Cu at (131.4, 120.5)
- added C17: 0.1uF, Capacitor_SMD:C_0402_1005Metric, F.Cu at (128.4, 103.2)
- added C2: 0.1uF, Capacitor_SMD:C_0402_1005Metric, F.Cu at (131.4, 117.8)
- added C3: 0.1uF, Capacitor_SMD:C_0402_1005Metric, F.Cu at (133.2, 107.4)
- added C4: 0.1uF, Capacitor_SMD:C_0402_1005Metric, F.Cu at (134.2, 107.4)
- added C5: 0.1uF, Capacitor_SMD:C_0402_1005Metric, F.Cu at (130.4, 104.3)
- added C6: 0.1uF, Capacitor_SMD:C_0402_1005Metric, F.Cu at (135.5, 109.8)
- added C7: 0.1uF, Capacitor_SMD:C_0402_1005Metric, F.Cu at (125.5, 109.0)
- added C8: 0.1uF, Capacitor_SMD:C_0402_1005Metric, F.Cu at (125.2, 113.5)
- added C9: 0.1uF, Capacitor_SMD:C_0402_1005Metric, F.Cu at (135.5, 113.5)
- added J1: USB_C_Receptacle_USB2.0_14P, Connector_USB:USB_C_Receptacle_HRO_TYPE-C-31-M-12, F.Cu at (130.5, 82.5)
- added J2: Conn_01x03, Connector_PinHeader_2.54mm:PinHeader_1x03_P2.54mm_Vertical, F.Cu at (128.0, 129.4)
- added J3: Conn_01x20, Connector_PinHeader_2.54mm:PinHeader_1x20_P2.54mm_Vertical, F.Cu at (121.6, 81.4)
- added J4: Conn_01x20, Connector_PinHeader_2.54mm:PinHeader_1x20_P2.54mm_Vertical, F.Cu at (139.4, 81.4)
- added R1: 5.1K, Resistor_SMD:R_0402_1005Metric, F.Cu at (128.8, 88.8)
- added R2: 5.1K, Resistor_SMD:R_0402_1005Metric, F.Cu at (131.8, 88.8)
- added R3: 27, Resistor_SMD:R_0402_1005Metric, F.Cu at (131.2, 107.4)
- added R4: 27, Resistor_SMD:R_0402_1005Metric, F.Cu at (132.2, 107.4)
- added R5: 1K, Resistor_SMD:R_0402_1005Metric, F.Cu at (128.9, 117.5)
- added R6: 1K, Resistor_SMD:R_0402_1005Metric, F.Cu at (134.4, 96.7)
- added R7: 10K, Resistor_SMD:R_0402_1005Metric, F.Cu at (126.5, 103.2)
- added SW1: SW_Push, Button_Switch_SMD:SW_Push_SPST_NO_Alps_SKRK, F.Cu at (134.3, 93.3)
- added U4: W25Q16JVZPIQ, Package_SON:Winbond_USON-8-1EP_3x2mm_P0.5mm_EP0.2x1.6mm, F.Cu at (127.3, 105.0)
- added Y1: Crystal_GND24, Crystal:Crystal_SMD_3225-4Pin_3.2x2.5mm_HandSoldering, F.Cu at (128.2, 120.5)
- U1: value NCP1117-1.5_SOT223 -> MCP1700x-330xxTT; footprint Package_TO_SOT_SMD:SOT-223-3_TabPin2 -> Package_TO_SOT_SMD:SOT-23
- moved U1 36.4 mm to (126.7, 91.5), turned to 90 degrees
- moved U2 21.2 mm to (130.3, 112.5)
Connections:
- U2 pad 20: USB_D+ -> XIN
- U2 pad 21: USB_D- -> XOUT

Commit message: PCB Designed!!!!!
Parts:
- removed C1: 1uF, Capacitor_SMD:C_0402_1005Metric
- removed C2: 0.1uF, Capacitor_SMD:C_0402_1005Metric
- added G***: LOGO, soup:soup!, B.Cu at (131.1, 99.2)
- moved J3 17.8 mm to (139.4, 81.4)
- moved J4 17.8 mm to (121.6, 81.4)
- moved C3 6.98 mm to (131.6, 100.7)
- moved C6 4.41 mm to (135.2, 105.5)
- moved C5 4.39 mm to (132.6, 100.5)
- moved R4 3.82 mm to (130.8, 103.8), turned to -90 degrees
- moved C11 3.77 mm to (130.5, 100.8)
- moved C17 3.60 mm to (128.5, 99.6), turned to 180 degrees
- moved R7 3.60 mm to (126.5, 99.6), turned to 180 degrees
- moved C7 3.60 mm to (125.7, 105.5), turned to 180 degrees
- moved U2 3.60 mm to (130.4, 109.0)
- moved U4 3.60 mm to (127.4, 101.4)
- moved R3 3.58 mm to (131.8, 103.9), turned to -90 degrees
- moved C4 3.58 mm to (133.8, 103.9)
- moved C10 3.57 mm to (132.9, 114.3), turned to -90 degrees
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Connections:
- C10 pad 1: +3V3 -> +1V1
- C11 pad 1: +3V3 -> +1V1
- C12 pad 1: +3V3 -> +1V1
- U2 pad 23: +3V3 -> +1V1
- U2 pad 43: +1V1 -> +3V3
- U2 pad 45: +3V3 -> +1V1
- U2 pad 48: +1V1 -> +3V3
- U2 pad 50: +3V3 -> +1V1
- U4 pad 4: unconnected-(U4-GND-Pad4) -> GND
- Y1 pad 1: XIN -> Net-(C16-Pad2)
- Y1 pad 3: Net-(C16-Pad2) -> XIN
Routing:
- net +3V3: track 0.00 -> 75.3 mm, vias 0 -> 8
- net GND: track 0.00 -> 41.3 mm, vias 0 -> 24
- net GPIO0: track 0.00 -> 30.2 mm, vias 0 -> 1
- net GPIO26_ADC3: track 0.00 -> 28.2 mm, vias 0 -> 2
- net +1V1: track 0.00 -> 26.5 mm, vias 0 -> 3
- net GPIO1: track 0.00 -> 26.0 mm, vias 0 -> 1
- net GPIO26_ADC2: track 0.00 -> 24.1 mm, vias 0 -> 2
- net GPIO15: track 0.00 -> 22.9 mm
- net USB_D-: track 0.00 -> 22.6 mm
- net USB_D+: track 0.00 -> 22.5 mm
- net SWCLK: track 0.00 -> 22.3 mm, vias 0 -> 1
- net GPIO16: track 0.00 -> 22.3 mm
- net GPIO2: track 0.00 -> 22.1 mm, vias 0 -> 1
- net VBUS: track 0.00 -> 20.4 mm
- net SWDIO: track 0.00 -> 20.3 mm, vias 0 -> 1
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- added copper zone on B.Cu, net GND
- added copper zone on F.Cu, net GND
Other:
- board text added: "Adhavan Diwakar Vidya"
- board text added: "Adithyan Diwakar Vidya"
- board text added: "AryanIndiaGavaskar"
- board text added: "Coimbatore Tamil Nadu, India"
- board text added: "Diwakar Raju"
- board text added: "Fallout"
- board text added: "Gavaskar Raju"
- board text added: "Nakshatra Gavaskar"
- board text added: "Parmimaladevi Raju"
- board text added: "Raju Chinnusamy"
- board text added: "Sarenya Gavaskar"
- board text added: "Vidya Diwakar"
