File: KiCad/ArxRP2040Devboard/ArxRP2040Devboard.kicad_sch (KiCad schematic)
At the start: 33 parts, among them J1 USB_C_Receptacle_USB2.0_14P, J2 Conn_01x03, J3 Conn_01x20, J4 Conn_01x20, SW1 SW_Push, U1 MCP1700x-330xxTT, U2 RP2040, U4 W25Q16JVZPIQ, Y1 Crystal_GND24

Commit message: gerber includes the position stuff
Parts:
- U4: Availability In Stock -> (none)
Changed lines of the file:
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@@
 			)
 		)
-		(property "Availability" "In Stock"
+		(property "AVAILABILITY" "In Stock"
 			(at 334.01 111.76 0)
 			(hide yes)
